File: ElectretXLRMic.kicad_pcb (KiCad board)
At the start: 2 copper layers, 37 x 51 mm, 38 parts, among them J1 MIC, J2 XLR3, U1 OPA1678

Commit message: Cleaned up DRC, some routing optimizations, geographical annotation
[KiCad Version: 10.0.1]
Parts:
- TP1: renamed from TP10; footprint TestPoint:TestPoint_Pad_2.5x2.5mm -> TestPoint:TestPoint_Pad_2.0x2.0mm
- TP10: renamed from TP9; footprint TestPoint:TestPoint_Pad_2.5x2.5mm -> TestPoint:TestPoint_Pad_2.0x2.0mm
- TP11: renamed from TP2; footprint TestPoint:TestPoint_Pad_2.5x2.5mm -> TestPoint:TestPoint_Pad_2.0x2.0mm
- TP2: renamed from TP11; footprint TestPoint:TestPoint_Pad_2.5x2.5mm -> TestPoint:TestPoint_Pad_2.0x2.0mm
- TP3: renamed from TP7; footprint TestPoint:TestPoint_Pad_2.5x2.5mm -> TestPoint:TestPoint_Pad_2.0x2.0mm
- TP4: renamed from TP3; footprint TestPoint:TestPoint_Pad_2.5x2.5mm -> TestPoint:TestPoint_Pad_2.0x2.0mm
- TP5: renamed from TP4; footprint TestPoint:TestPoint_Pad_2.5x2.5mm -> TestPoint:TestPoint_Pad_2.0x2.0mm
- TP6: renamed from TP1; footprint TestPoint:TestPoint_Pad_2.5x2.5mm -> TestPoint:TestPoint_Pad_2.0x2.0mm
- TP7: renamed from TP5; footprint TestPoint:TestPoint_Pad_2.5x2.5mm -> TestPoint:TestPoint_Pad_2.0x2.0mm
- TP8: renamed from TP6; footprint TestPoint:TestPoint_Pad_2.5x2.5mm -> TestPoint:TestPoint_Pad_2.0x2.0mm
- TP9: renamed from TP8; footprint TestPoint:TestPoint_Pad_2.5x2.5mm -> TestPoint:TestPoint_Pad_2.0x2.0mm
- moved TP11 0.50 mm to (122.0, 63.5)
- renumbered C6 to C1, C5 to C10, C3 to C2, C10 to C3, C7 to C4, C1 to C5, C9 to C6, C4 to C7, C2 to C8, C8 to C9, D3 to D1, D1 to D2, D2 to D3, H2 to H1, H1 to H2, J2 to J1, J1 to J2, R5 to R1, R6 to R2, R2 to R3, R8 to R4, R3 to R5, R9 to R6, R4 to R7, R7 to R8, R1 to R9
Connections:
- net +IN_A renamed Net-(J2-Pin_1)
- net +IN_B renamed Net-(C2-+)
- net -IN_A renamed Net-(U1A--)
- net -IN_B renamed Net-(U1B--)
- net OUT_B renamed Net-(C4-Pad1)
- net V+ renamed Net-(U1C-V+)
- net V- renamed GND
Routing:
- net Net-(U1C-V+): track 41.6 -> 41.0 mm
- net GND: vias 227 -> 235
