File: ElectretXLRMic.kicad_sch (KiCad schematic)
At the start: 51 parts, among them IC1 OPA1678IDR, J1 MIC, J2 XLR3, J3 XLR3, U1 OPA1678

Commit message: Readme update/test Slight changes to the schematic
[KiCad Version: 9.0.7]
Other:
- note added: "Do not use ceramic caps from X or Y series for signals. Capacitors should be rated for >=63 VDC Buy 2x of everything DC voltage at TP U1A+ should be half of VCC (or atleast between 3.5 V-4.7 V) ! Change R2 value. Change R1 value to a larger one up to 330 Ohm if not clipping when R2 is balanced."
- note removed: "Do not use ceramic caps from X or Y series for signals. Capacitors should be rated for >=63 VDC Buy 2x of everything Match the 33uF DC blocking caps (C12, C13) as close as possible with a multimeter/LCR meter DC voltage at TP U1A+ should be 4.1 V (or atleast between 3.5 V-4.7 V) ! Change R2 value. Change R1 value to a larger one up to 330 Ohm if not clipping when R2 is balanced."
Changed lines of the file:
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@@
 		(rev "1.1")
 	)
-	(text "Do not use ceramic caps from X or Y series for signals.\nCapacitors should be rated for >=63 VDC\nBuy 2x of everything\nMatch the 33uF DC blocking caps (C12, C13) as close as possible with a multimeter/LCR meter\nDC voltage at TP U1A+ should be 4.1 V (or atleast between 3.5 V-4.7 V) ! Change R2 value.\n\nChange R1 value to a larger one up to 330 Ohm if not clipping when R2 is balanced."
+	(text "Do not use ceramic caps from X or Y series for signals.\nCapacitors should be rated for >=63 VDC\nBuy 2x of everything\nDC voltage at TP U1A+ should be half of VCC (or atleast between 3.5 V-4.7 V) ! Change R2 value.\n\nChange R1 value to a larger one up to 330 Ohm if not clipping when R2 is balanced."
 		(exclude_from_sim no)
 		(at 89.916 36.322 0)

Commit message: The TVS diodes had slightly different footprints, fixed now.
[KiCad Version: 9.0.7]
Parts:
- D2: footprint Diode_SMD:D_SMA -> Diode_SMD:D_SMA_Handsoldering
Changed lines of the file:
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@@
 			)
 		)
-		(property "Footprint" "Diode_SMD:D_SMA"
+		(property "Footprint" "Diode_SMD:D_SMA_Handsoldering"
 			(at 193.04 82.55 0)
 			(effects

Commit message: Test of the circuit is done and final adjustments done for values. BOM has reduced amount of resistors and capacitors. Added 2.54 mm pitch wire terminals to BOM because getting the wires to the connectors was a pain.
[KiCad Version: 9.0.7]
Parts:
- removed C11, C12, C13: 33uF, Capacitor_SMD:C_Elec_8x10.2, symbol Device:C_Polarized
- removed H2: MountingHole_Pad, MountingHole:MountingHole_2.7mm_M2.5_DIN965_Pad_TopBottom, symbol Mechanical:MountingHole_Pad
- removed IC1: OPA1678IDR, SamacSys_Parts:SOIC127P600X175-8N, symbol SamacSys_Parts:OPA1678IDR
- removed R10: 4.7k, Resistor_SMD:R_0603_1608Metric_Pad0.98x0.95mm_HandSolder, symbol Device:R
- removed R11: 5.6k, Resistor_SMD:R_0603_1608Metric_Pad0.98x0.95mm_HandSolder, symbol Device:R
- removed R12: 8.2k, Resistor_SMD:R_0603_1608Metric_Pad0.98x0.95mm_HandSolder, symbol Device:R
- removed R13: 10k, Resistor_SMD:R_0603_1608Metric_Pad0.98x0.95mm_HandSolder, symbol Device:R
- removed R14: 12k, Resistor_SMD:R_0603_1608Metric_Pad0.98x0.95mm_HandSolder, symbol Device:R
- removed R15: 15k, Resistor_SMD:R_0603_1608Metric_Pad0.98x0.95mm_HandSolder, symbol Device:R
- removed R16: 220, Resistor_SMD:R_0603_1608Metric_Pad0.98x0.95mm_HandSolder, symbol Device:R
- removed R17: 100, Resistor_SMD:R_0603_1608Metric_Pad0.98x0.95mm_HandSolder, symbol Device:R
- added H2: MountingHole, MountingHole:MountingHole_2.5mm, symbol Mechanical:MountingHole
- H1: value MountingHole_Pad -> MountingHole_GND
- J1: Manufacturer_Part_Number (none) -> TBC05-02-1-G-G; now in the parts list
- J2: Manufacturer_Part_Number (none) -> TBC05-03-1-G-G; now in the parts list
- R1: renamed from R2; value 6.8k -> 7.5k; Manufacturer_Part_Number CRT0603ABY-6801ELF -> ERA-1AEB752C
- U1: footprint (none) -> Package_SO:SOIC-8_3.9x4.9mm_P1.27mm; Manufacturer_Part_Number (none) -> OPA1678IDR; now in the parts list
- renumbered C6 to C1, C7 to C10, C1 to C2, C10 to C3, C2 to C4, C3 to C5, C5 to C6, C9 to C7, C4 to C8, C8 to C9, D3 to D2, D2 to D3, R6 to R2, R7 to R3, R8 to R4, R9 to R6, R1 to R7, R3 to R8, R4 to R9, TP7 to TP1, TP5 to TP10, TP6 to TP11, TP1 to TP2, TP8 to TP3, TP10 to TP4, TP2 to TP5, TP3 to TP6, TP9 to TP7, TP11 to TP8, TP4 to TP9
Connections:
- no-connect marks 1 -> 0
Other:
- note added: "Do not use ceramic caps from X or Y series for signals. Capacitors should be rated for >=63 VDC"
- note added: "Electret bias voltage should be close to 3.4 V. The value of the resistor depends on the mic capsule/the JFET."
- note added: "Voltage after R7 is approx 6.8 V"
- note removed: "Do not use ceramic caps from X or Y series for signals. Capacitors should be rated for >=63 VDC Buy 2x of everything DC voltage at TP U1A+ should be half of VCC (or atleast between 3.5 V-4.7 V) ! Change R2 value. Change R1 value to a larger one up to 330 Ohm if not clipping when R2 is balanced."
- moved on the sheet: C1, C10, C2, C3, C4, C5, C6, C7, C8, C9, D1, D2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

Commit message: Cleaned up DRC, some routing optimizations, geographical annotation
[KiCad Version: 10.0.1]
Parts:
- D1: renamed from D3; footprint Diode_SMD:D_SMA_Handsoldering -> Diode_SMD:D_SMA
- D3: renamed from D2; footprint Diode_SMD:D_SMA_Handsoldering -> Diode_SMD:D_SMA
- renumbered C6 to C1, C5 to C10, C3 to C2, C10 to C3, C7 to C4, C1 to C5, C9 to C6, C4 to C7, C2 to C8, C8 to C9, D1 to D2, H2 to H1, H1 to H2, J2 to J1, J1 to J2, R5 to R1, R6 to R2, R2 to R3, R8 to R4, R3 to R5, R9 to R6, R4 to R7, R7 to R8, R1 to R9, TP10 to TP1, TP9 to TP10, TP2 to TP11, TP11 to TP2, TP7 to TP3, TP3 to TP4, TP4 to TP5, TP1 to TP6, TP5 to TP7, TP6 to TP8, TP8 to TP9
Connections:
- net +IN_A: no longer names the net of C5.1, J2.1 (Pin_1), R9.2, TP6.1, U1.3 (+)
- net +IN_B: no longer names the net of C2.1 (+), R3.2, U1.5 (+)
- net -IN_A: no longer names the net of C1.2, R3.1, R5.1, TP4.1, U1.1, U1.2 (-)
- net -IN_B: no longer names the net of R5.2, R7.1, U1.6 (-)
- net OUT_B: no longer names the net of C4.1, R7.2, TP5.1, U1.7
- net V+: no longer names the net of C10.1, C7.1, C8.1, C9.1, R8.2, R9.1, TP11.1, U1.8 (V+)
Other:
- moved on the sheet: TP11
